File: Map/lsu/lsu.sch (KiCad schematic (older format))
At the start: 0 parts

Commit message: Release v1
Changed lines of the file:
@@
 $EndSheet
 $Sheet
-S 4300 1550 600  650
+S 4200 1650 650  600
 U 5EA99702
 F0 "C2" 50
 F1 "Mullers_gate.sch" 50
-F2 "req_in" I T 4800 1550 50
-F3 "ack_in" I B 4400 2200 50
-F4 "req_o" O B 4800 2200 50
+F2 "req_in" I L 4200 1750 50
+F3 "ack_in" I R 4850 2150 50
+F4 "req_o" O R 4850 1750 50
 $EndSheet
 $Sheet

Commit message: screen
Connections:
- no-connect marks 2 -> 0
Changed lines of the file:
@@
 $EndSheet
 $Sheet
-S 4050 2750 1150 2100
+S 4050 2750 1100 450
 U 5EA999FC
 F0 "DM" 50
@@
 F3 "data_we_i" I L 4050 2900 50
 F4 "data_wdata_i" I L 4050 3000 50
-F5 "data_rdata_o" O R 5200 2900 50
-F6 "data_err_o" O R 5200 3000 50
-F7 "req" I L 4050 2800 50
+F5 "data_rdata_o" O R 5150 2900 50
+F6 "data_err_o" O R 5150 3000 50
+F7 "en" I L 4050 2800 50
 $EndSheet
 Wire Wire Line
@@
 	2450 1750 2850 1750
 $Sheet
-S 6450 2750 1150 600
+S 6450 2750 1150 450
 U 5EA99C84
 F0 "lsu_out" 50
@@
 F3 "data_err_i" I L 6450 3000 50
 F4 "lsu_rdata_o" O R 7600 2900 50
-F5 "req" I L 6450 2800 50
+F5 "en" I L 6450 2800 50
 F6 "lsu_err_o" O R 7600 3000 50
 $EndSheet
@@
 	4850 2150 6000 2150
 $Sheet
-S 2100 2750 1400 2100
+S 2100 2750 1350 450
 U 5EA99C56
 F0 "lsu_in" 50
 F1 "LSU_in.sch" 50
-F2 "data_addr_o" O R 3500 3100 50
-F3 "data_we_o" O R 3500 2900 50
-F4 "data_wdata_o" O R 3500 3000 50
+F2 "data_addr_o" O R 3450 3100 50
+F3 "data_we_o" O R 3450 2900 50
+F4 "data_wdata_o" O R 3450 3000 50
 F5 "lsu_we_i" I L 2100 2900 50
 F6 "lsu_wdata_i" I L 2100 3000 50
 F7 "adder_result_ex_i" I L 2100 3100 50
-F8 "req" I L 2100 2800 50
+F8 "en" I L 2100 2800 50
 $EndSheet
 Text Label 2500 1750 0    50   ~ 0
@@
 Connection ~ 3650 2500
 Wire Wire Line
-	3500 2900 4050 2900
-Wire Wire Line
-	3500 3000 4050 3000
-Wire Wire Line
-	3500 3100 4050 3100
-Wire Wire Line
 	4050 2800 4000 2800
 Wire Wire Line
@@
 Wire Wire Line
 	4000 2500 3800 2500
-NoConn ~ 4000 2650
-Wire Wire Line
-	5200 2900 6450 2900
-Wire Wire Line
-	5200 3000 6450 3000
 Wire Wire Line
 	6450 2800 6000 2800
@@
 	6000 2800 6000 2550
 Connection ~ 6000 2550
-NoConn ~ 5550 2150
+Wire Wire Line
+	3450 2900 4050 2900
+Wire Wire Line
+	3450 3000 4050 3000
+Wire Wire Line
+	3450 3100 4050 3100
+Wire Wire Line
+	5150 2900 6450 2900
+Wire Wire Line
+	5150 3000 6450 3000
 $EndSCHEMATC
